File: circuit/wht.kicad_pcb (KiCad board)
At the start: 2 copper layers, 50 x 44 mm, 18 parts, among them M1 NRF24LE1_SMALL, Q1 TPS1101D, SW1 SW_PUSH, SW2 SWITCH_INV, U1 NRF24LE1_PROG, U2 MPU-6050, U3 UART

Commit message: - fixed a problem with the circuit project file; added library references - changed the project address on the bottom of the PCB
Other:
- board text added: "Wireless Head Tracker http://wireless-head-tracker.googlecode.com/ Based on ED Tracker http://edtracker.org.uk/"
- board text removed: "Wireless Head Tracker https://code.google.com/p/wireless-head-tracker/ Based on ED Tracker http://edtracker.org.uk/"
